Commit message: 修改urdf为新机器人

File: tita_rl-master/resources/tita/urdf/tita_description.urdf (robot description, URDF)
Before this commit: robot tita_ros2_control, 14 links, 13 joints
Links:
- link base_link: mass 13.2 -> 18.96; geometry collision mesh filename=../meshes/base_link.STL; visual mesh filename=../meshes/base_link.STL
- link left_leg_1: mass 2.064 -> 4.65; geometry visual mesh filename=../meshes/L_1.STL
- link left_leg_2: mass 3.0984 -> 3.14; geometry visual mesh filename=../meshes/L_2.STL
- link left_leg_3: mass 0.57244 -> 1.59; geometry collision box size=0.28 0.07 0.02; visual mesh filename=../meshes/L_3.STL
- link left_leg_4: mass 1.5094 -> 1.54; geometry collision cylinder length=0.03 radius=0.09; visual mesh filename=../meshes/L_4.STL
- link right_leg_1: mass 2.064 -> 4.65; geometry visual mesh filename=../meshes/R_1.STL
- link right_leg_2: mass 3.0987 -> 3.14; geometry visual mesh filename=../meshes/R_2.STL
- link right_leg_3: mass 0.57244 -> 1.59; geometry collision box size=0.28 0.07 0.02; visual mesh filename=../meshes/R_3.STL
- link right_leg_4: mass 1.5094 -> 1.54; geometry collision cylinder length=0.03 radius=0.09; visual mesh filename=../meshes/R_4.STL
Joints:
- joint joint_left_leg_1: limit lower=-0.785398 upper=0.785398 effort=60 velocity=25 -> lower=-1.5708 upper=1.5708 effort=60 velocity=15; origin xyz=0 0.0895 0 rpy=1.5708 0 1.5708 -> xyz=0 0.131 0 rpy=1.5776 -2.4621E-05 1.5708
- joint joint_left_leg_2: limit lower=-1.919862 upper=3.490659 effort=60 velocity=25 -> lower=-1.919 upper=2.618 effort=60 velocity=15; origin xyz=0.1426 0 0 rpy=-1.5708 0 -1.5708 -> xyz=0.1264 0 0 rpy=-1.5708 -0.086165 -1.5708
- joint joint_left_leg_3: limit lower=-2.670354 upper=-0.698132 effort=60 velocity=25 -> lower=-2.3562 upper=-0.7854 effort=60 velocity=15; origin xyz=0.2 0 0 rpy=0 0 0 -> xyz=0.25 0 0 rpy=0 0 0.072636
- joint joint_left_leg_4: limit lower=-999999 upper=999999 effort=15 velocity=20 -> lower=-999999 upper=999999 effort=7 velocity=20; origin xyz=0.2 0 0.0514 rpy=0 0 0 -> xyz=0.22 0 0.0581 rpy=0 0 -1.5573
- joint joint_right_leg_1: axis 0 0 1 -> 0 0 -1; limit lower=-0.785398 upper=0.785398 effort=60 velocity=25 -> lower=-1.5708 upper=1.5708 effort=60 velocity=15; origin xyz=0 -0.0895 0 rpy=1.5708 0 1.5708 -> xyz=0 -0.131 -1.2901E-05 rpy=1.5776 -2.4621E-05 1.5708
- joint joint_right_leg_2: limit lower=-1.919862 upper=3.490659 effort=60 velocity=25 -> lower=-1.919 upper=2.618 effort=60 velocity=15; origin xyz=-0.1426 0 0 rpy=-1.5708 0 -1.5708 -> xyz=-0.1264 0 0 rpy=-1.5708 -0.086869 -1.5708
- joint joint_right_leg_3: limit lower=-2.670354 upper=-0.698132 effort=60 velocity=25 -> lower=-2.3562 upper=-0.7854 effort=60 velocity=15; origin xyz=0.2 0 0 rpy=0 0 0 -> xyz=0.25 0 0 rpy=0 0 0.074137
- joint joint_right_leg_4: limit lower=-999999 upper=999999 effort=15 velocity=20 -> lower=-999999 upper=999999 effort=7 velocity=20; origin xyz=0.2 0 -0.0514 rpy=0 0 0 -> xyz=0.22 0 -0.05845 rpy=0 0 -1.5581
